File: watch_pcb.kicad_sch (KiCad schematic)
At the start: 22 parts, among them Q1 AO3400A, Q2 AO3400A, Q3 AO3400A, Q4 AO3400A, U1 JSS-3941AUW-21, U2 ATtiny3217-M

Commit message: Slight modification to schematic
Connections:
- net PA7: now reaches U2.8 (PA7)
- net PA7: now also R17.2
- net PA6: no longer names the net of U2.7 (PA6)
- net PA6: no longer R17.2
Changed lines of the file:
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@@
 		)
 	)
-	(label "PA6"
+	(label "PA7"
 		(at 115.57 83.82 0)
 		(effects
@@
 		)
 	)
-	(label "PA6"
-		(at 246.38 50.8 0)
+	(label "PA7"
+		(at 246.38 53.34 0)
 		(effects
 			(font

Commit message: Modified schematic
Parts:
- added C1, C2: 8.2pF, symbol Device:C
- added Y1: 32.768kHz, symbol Device:Crystal
Connections:
- net GND: now also C1.2, C2.2
- net SEG_C: now also U2.18 (PC1); no longer U2.14 (PB2)
- net SEG_COL: now also U2.22 (PC5); no longer U2.10 (PB6)
- net SEG_D: now also U2.19 (PC2); no longer U2.13 (PB3)
- net SEG_E: now also U2.20 (PC3); no longer U2.12 (PB4)
- net SEG_F: now also U2.21 (PC4); no longer U2.11 (PB5)
- new net: C2.1, U2.13 (PB3), Y1.1
- new net: C1.1, U2.14 (PB2), Y1.2
